Commit message: 更新 U 盘模型代码7121027

File: urdf/URDFzhuangpei.SLDASM.urdf (robot description, URDF)
Before this commit: robot URDFzhuangpei.SLDASM, 14 links, 13 joints
Links:
- added link FL_foot, mass 0.01; collision sphere radius=0.016; visual sphere radius=0.015
- added link FR_foot, mass 0.01; collision sphere radius=0.016; visual sphere radius=0.015
- added link RL_foot, mass 0.01; collision sphere radius=0.016; visual sphere radius=0.015
- added link RR_foot, mass 0.01; collision sphere radius=0.016; visual sphere radius=0.015
- link FL_calf_joint: mass 0.23404332064939 -> 0.14; geometry collision cylinder length=0.023 radius=0.020; collision cylinder length=0.04 radius=0.011
- link FL_hip_joint: geometry collision box size=0.028 0.068 0.064; collision cylinder length=0.04 radius=0.038
- link FL_thigh_joint: mass 0.872150809470834 -> 0.8; geometry collision box size=0.028 0.024 0.095; visual mesh filename=package://URDFzhuangpei.SLDASM/meshes/FL_thigh_joint.STL
- link FR_calf_joint: mass 0.234042505684366 -> 0.14; geometry collision cylinder length=0.023 radius=0.020; collision cylinder length=0.04 radius=0.011
- link FR_hip_joint: geometry collision box size=0.028 0.068 0.064; collision cylinder length=0.04 radius=0.038
- link FR_thigh_joint: mass 0.872150153156901 -> 0.8; geometry collision box size=0.028 0.024 0.095; visual mesh filename=package://URDFzhuangpei.SLDASM/meshes/FR_thigh_joint.STL
- link RL_calf_joint: mass 0.23404332064939 -> 0.14; geometry collision cylinder length=0.023 radius=0.020; collision cylinder length=0.04 radius=0.011
- link RL_hip_joint: geometry collision box size=0.028 0.068 0.064; collision cylinder length=0.04 radius=0.038
- link RL_thigh_joint: mass 0.872150809470864 -> 0.8; geometry collision box size=0.028 0.024 0.095; visual mesh filename=package://URDFzhuangpei.SLDASM/meshes/RL_thigh_joint.STL
- link RR_calf_joint: mass 0.234042505684366 -> 0.14; geometry collision cylinder length=0.023 radius=0.020; collision cylinder length=0.04 radius=0.011
- link RR_hip_joint: geometry collision box size=0.028 0.068 0.064; collision cylinder length=0.04 radius=0.038
- link RR_thigh_joint: mass 0.872150152908066 -> 0.8; geometry collision box size=0.028 0.024 0.095; visual mesh filename=package://URDFzhuangpei.SLDASM/meshes/RR_thigh_joint.STL
- link Trunk: mass 4.35129728273739 -> 5.2; geometry collision box size=0.082 0.215 0.095; collision box size=0.082 0.215 0.095
- link imu_Link: geometry collision box size=0.03 0.02 0.002; visual mesh filename=package://URDFzhuangpei.SLDASM/meshes/imu_Link.STL
Joints:
- added joint FL_foot_fixed: type fixed, parent FL_calf_joint, child FL_foot, origin xyz=0.201984878571 0 0.00837310150402 rpy=0 0 0
- added joint FR_foot_fixed: type fixed, parent FR_calf_joint, child FR_foot, origin xyz=0.201984878568 0 0.00837310156582 rpy=0 0 0
- added joint RL_foot_fixed: type fixed, parent RL_calf_joint, child RL_foot, origin xyz=0.201984876549 0 0.00837315026116 rpy=0 0 0
- added joint RR_foot_fixed: type fixed, parent RR_calf_joint, child RR_foot, origin xyz=0.201984876547 0 0.0083731503174 rpy=0 0 0
- joint FL_calf_joint: limit lower=0 upper=0 effort=0 velocity=0 -> lower=0 upper=1.91986217719 effort=17 velocity=32.9867
- joint FL_hip_joint: axis 0 1 0 -> 1 0 0; limit lower=0 upper=0 effort=0 velocity=0 -> lower=-1.0472 upper=1.0472 effort=17 velocity=32.9867
- joint FL_thigh_joint: limit lower=0 upper=0 effort=0 velocity=0 -> lower=-2.76228694714 upper=2.29921305286 effort=17 velocity=32.9867
- joint FR_calf_joint: limit lower=0 upper=0 effort=0 velocity=0 -> lower=-1.91986217719 upper=0 effort=17 velocity=32.9867
- joint FR_hip_joint: axis 0 -1 0 -> 1 0 0; limit lower=0 upper=0 effort=0 velocity=0 -> lower=-1.0472 upper=1.0472 effort=17 velocity=32.9867
- joint FR_thigh_joint: limit lower=0 upper=0 effort=0 velocity=0 -> lower=-2.29921305286 upper=2.76228694714 effort=17 velocity=32.9867
- joint RL_calf_joint: limit lower=0 upper=0 effort=0 velocity=0 -> lower=0 upper=1.91986217719 effort=17 velocity=32.9867
- joint RL_hip_joint: axis 0 1 0 -> 1 0 0; limit lower=0 upper=0 effort=0 velocity=0 -> lower=-1.0472 upper=1.0472 effort=17 velocity=32.9867
- joint RL_thigh_joint: limit lower=0 upper=0 effort=0 velocity=0 -> lower=-2.76228694714 upper=2.29921305286 effort=17 velocity=32.9867
- joint RR_calf_joint: limit lower=0 upper=0 effort=0 velocity=0 -> lower=-1.91986217719 upper=0 effort=17 velocity=32.9867
- joint RR_hip_joint: axis 0 -1 0 -> 1 0 0; limit lower=0 upper=0 effort=0 velocity=0 -> lower=-1.0472 upper=1.0472 effort=17 velocity=32.9867
- joint RR_thigh_joint: limit lower=0 upper=0 effort=0 velocity=0 -> lower=-2.29921305286 upper=2.76228694714 effort=17 velocity=32.9867

Commit message: 更新 U 盘模型代码7211549

File: urdf/URDFzhuangpei.SLDASM.urdf (robot description, URDF)
Before this commit: robot URDFzhuangpei.SLDASM, 18 links, 17 joints
Joints:
- joint FR_calf_joint: axis 0 -1 0 -> 0 1 0; limit lower=-1.91986217719 upper=0 effort=17 velocity=32.9867 -> lower=0 upper=1.91986217719 effort=17 velocity=32.9867
- joint FR_thigh_joint: axis 0 -1 0 -> 0 1 0; limit lower=-2.29921305286 upper=2.76228694714 effort=17 velocity=32.9867 -> lower=-2.76228694714 upper=2.29921305286 effort=17 velocity=32.9867
- joint RR_calf_joint: axis 0 -1 0 -> 0 1 0; limit lower=-1.91986217719 upper=0 effort=17 velocity=32.9867 -> lower=0 upper=1.91986217719 effort=17 velocity=32.9867
- joint RR_thigh_joint: axis 0 -1 0 -> 0 1 0; limit lower=-2.29921305286 upper=2.76228694714 effort=17 velocity=32.9867 -> lower=-2.76228694714 upper=2.29921305286 effort=17 velocity=32.9867
